Commit message: Fixed dependencies

File: arm7dof/arm7dof_model/arm7dof_model.xacro (robot description, xacro)
@@ -338,5 +338,5 @@
   <transmission name="tran7">
 	<type>transmission_interface/SimpleTransmission</type>
-	<joint name="ft_sensor_jnt">
+	<joint name="wrench">
 	  <!--hardwareInterface>PositionJointInterface</hardwareInterface-->
 	  <!--hardwareInterface>VelocityJointInterface</hardwareInterface-->
@@ -356,15 +356,15 @@
   </gazebo>
   <!--model a f/t sensor; set up a link and a joint -->
-  <link name="ft_sensor_link">
+  <link name="wrench">
       <collision>
           <origin xyz="0 0 ${-L_flange_disk/2}" rpy="0 0 0"/>
           <geometry>
-            <cylinder length="${L_flange_disk}" radius="${r_endplate}"/>
-          </geometry>
+            <mesh filename="file:///home/user/ros_ws/src/socket_wrench.stl"  scale="0.05 0.05 0.05"/>
+        </geometry>
       </collision>
       <visual>
           <origin xyz="0 0 ${-L_flange_disk/2}" rpy="0 0 0" />
           <geometry>
-              <cylinder length="${L_flange_disk}" radius="${r_endplate}"/>
+            <mesh filename="file:///home/user/ros_ws/src/socket_wrench.stl"  scale="0.05 0.05 0.05"/>
           </geometry>
           <material name="ft_sensor_color">
@@ -379,8 +379,8 @@
   </link>
   <!--ideally, this would be a static joint; until fixed in gazebo, must have dynamic jnt-->
-  <joint name="ft_sensor_jnt" type="prismatic">
+  <joint name="wrench_jnt" type="prismatic">
     <parent link="link8"/>
-    <child link="ft_sensor_link"/>
-    <origin xyz="0 0 -0.003" rpy="0 0 0"/>
+    <child link="wrench"/>
+    <origin xyz="-0.85 0 -0.003" rpy="1.57 0 0"/>
     <axis xyz="0 0 1"/>
     <limit effort="100.0" lower="0" upper="0.0" velocity="0.01"/>
@@ -388,14 +388,3 @@
   </joint>
     <!-- Enable Joint Feedback -->
-    <gazebo reference="ft_sensor_jnt">
-        <provideFeedback>true</provideFeedback>
-    </gazebo>
-    <!-- The ft_sensor plugin -->
-    <gazebo>
-        <plugin name="ft_sensor" filename="libgazebo_ros_ft_sensor.so">
-            <updateRate>1000.0</updateRate>
-            <topicName>ft_sensor_topic</topicName>
-            <jointName>ft_sensor_jnt</jointName>
-        </plugin>
-    </gazebo>
 </robot>

Commit message: More fixes needed

File: arm7dof/arm7dof_model/arm7dof_model.xacro (robot description, xacro)
@@ -338,5 +338,5 @@
   <transmission name="tran7">
 	<type>transmission_interface/SimpleTransmission</type>
-	<joint name="wrench">
+	<joint name="wrench_jnt">
 	  <!--hardwareInterface>PositionJointInterface</hardwareInterface-->
 	  <!--hardwareInterface>VelocityJointInterface</hardwareInterface-->
@@ -360,5 +360,5 @@
           <origin xyz="0 0 ${-L_flange_disk/2}" rpy="0 0 0"/>
           <geometry>
-            <mesh filename="file:///home/user/ros_ws/src/socket_wrench.stl"  scale="0.05 0.05 0.05"/>
+            <mesh filename="file:///home/user/ros_ws/src/Loose-screw/socket_wrench.stl"  scale="0.05 0.05 0.05"/>
         </geometry>
       </collision>
@@ -366,5 +366,5 @@
           <origin xyz="0 0 ${-L_flange_disk/2}" rpy="0 0 0" />
           <geometry>
-            <mesh filename="file:///home/user/ros_ws/src/socket_wrench.stl"  scale="0.05 0.05 0.05"/>
+            <mesh filename="file:///home/user/ros_ws/src/Loose-screw/socket_wrench.stl"  scale="0.05 0.05 0.05"/>
           </geometry>
           <material name="ft_sensor_color">

Commit message: Updated robot model
Changed the transmissions on the robot model to accommodate new control mechanism

File: arm7dof/arm7dof_model/arm7dof_model.xacro (robot description, xacro)
@@ -237,116 +237,76 @@
 	</inertial>
   </link>
-  <transmission name="tran0">
-	<type>transmission_interface/SimpleTransmission</type>
-	<joint name="joint0">
-	  <!--hardwareInterface>PositionJointInterface</hardwareInterface-->
-	  <!--hardwareInterface>VelocityJointInterface</hardwareInterface-->
-	  <hardwareInterface>EffortJointInterface</hardwareInterface>
-	</joint>
-	<actuator name="motor0">
-	  <!--hardwareInterface>PositionJointInterface</hardwareInterface-->
-	  <!--hardwareInterface>VelocityJointInterface</hardwareInterface-->
-	  <hardwareInterface>EffortJointInterface</hardwareInterface>
-	  <mechanicalReduction>7680</mechanicalReduction>
-	</actuator>
+<transmission name="tran0">
+    <type>transmission_interface/SimpleTransmission</type>
+    <joint name="joint0">
+      <hardwareInterface>hardware_interface/PositionJointInterface</hardwareInterface>
+    </joint>
+    <actuator name="motor0">
+      <mechanicalReduction>7680</mechanicalReduction>
+    </actuator>
   </transmission>
   <transmission name="tran1">
-	<type>transmission_interface/SimpleTransmission</type>
-	<joint name="joint1">
-	  <!--hardwareInterface>PositionJointInterface</hardwareInterface-->
-	  <!--hardwareInterface>VelocityJointInterface</hardwareInterface-->
-	  <hardwareInterface>EffortJointInterface</hardwareInterface>
-	</joint>
-	<actuator name="motor1">
-	  <!--hardwareInterface>PositionJointInterface</hardwareInterface-->
-	  <!--hardwareInterface>VelocityJointInterface</hardwareInterface-->
-	  <hardwareInterface>EffortJointInterface</hardwareInterface>
-	  <mechanicalReduction>7680</mechanicalReduction>
-	</actuator>
+    <type>transmission_interface/SimpleTransmission</type>
+    <joint name="joint1">
+      <hardwareInterface>hardware_interface/PositionJointInterface</hardwareInterface>
+    </joint>
+    <actuator name="motor1">
+      <mechanicalReduction>7680</mechanicalReduction>
+    </actuator>
   </transmission>
   <transmission name="tran2">
-	<type>transmission_interface/SimpleTransmission</type>
-	<joint name="joint2">
-	  <!--hardwareInterface>PositionJointInterface</hardwareInterface-->
-	  <!--hardwareInterface>VelocityJointInterface</hardwareInterface-->
-	  <hardwareInterface>EffortJointInterface</hardwareInterface>
-	</joint>
-	<actuator name="motor2">
-	  <!--hardwareInterface>PositionJointInterface</hardwareInterface-->
-	  <!--hardwareInterface>VelocityJointInterface</hardwareInterface-->
-	  <hardwareInterface>EffortJointInterface</hardwareInterface>
-	  <mechanicalReduction>3584</mechanicalReduction>
-	</actuator>
+    <type>transmission_interface/SimpleTransmission</type>
+    <joint name="joint2">
+      <hardwareInterface>hardware_interface/PositionJointInterface</hardwareInterface>
+    </joint>
+    <actuator name="motor2">
+      <mechanicalReduction>3584</mechanicalReduction>
+    </actuator>
   </transmission>
   <transmission name="tran3">
-	<type>transmission_interface/SimpleTransmission</type>
-	<joint name="joint3">
-	  <!--hardwareInterface>PositionJointInterface</hardwareInterface-->
-	  <!--hardwareInterface>VelocityJointInterface</hardwareInterface-->
-	  <hardwareInterface>EffortJointInterface</hardwareInterface>
-	</joint>
-	<actuator name="motor3">
-	  <!--hardwareInterface>PositionJointInterface</hardwareInterface-->
-	  <!--hardwareInterface>VelocityJointInterface</hardwareInterface-->
-	  <hardwareInterface>EffortJointInterface</hardwareInterface>
-	  <mechanicalReduction>3584</mechanicalReduction>
-	</actuator>
-  </transmission>
-  <transmission name="tran4">
-	<type>transmission_interface/SimpleTransmission</type>
-	<joint name="joint4">
-	  <!--hardwareInterface>PositionJointInterface</hardwareInterface-->
-	  <!--hardwareInterface>VelocityJointInterface</hardwareInterface-->
-	  <hardwareInterface>EffortJointInterface</hardwareInterface>
-	</joint>
-	<actuator name="motor4">
-	  <!--hardwareInterface>PositionJointInterface</hardwareInterface-->
-	  <!--hardwareInterface>VelocityJointInterface</hardwareInterface-->
-	  <hardwareInterface>EffortJointInterface</hardwareInterface>
-	  <mechanicalReduction>3125</mechanicalReduction>
-	</actuator>
+    <type>transmission_interface/SimpleTransmission</type>
+    <joint name="joint3">
+      <hardwareInterface>hardware_interface/PositionJointInterface</hardwareInterface>
+    </joint>
+    <actuator name="motor3">
+      <mechanicalReduction>3584</mechanicalReduction>
+    </actuator>
+  </transmission>
+ <transmission name="tran4">
+    <type>transmission_interface/SimpleTransmission</type>
+    <joint name="joint4">
+      <hardwareInterface>hardware_interface/PositionJointInterface</hardwareInterface>
+    </joint>
+    <actuator name="motor4">
+      <mechanicalReduction>3125</mechanicalReduction>
+    </actuator>
   </transmission>
   <transmission name="tran5">
-	<type>transmission_interface/SimpleTransmission</type>
-	<joint name="joint5">
-	  <!--hardwareInterface>PositionJointInterface</hardwareInterface-->
-	  <!--hardwareInterface>VelocityJointInterface</hardwareInterface-->
-	  <hardwareInterface>EffortJointInterface</hardwareInterface>
-	</joint>
-	<actuator name="motor5">
-	  <!--hardwareInterface>PositionJointInterface</hardwareInterface-->
-	  <!--hardwareInterface>VelocityJointInterface</hardwareInterface-->
-	  <hardwareInterface>EffortJointInterface</hardwareInterface>
-	  <mechanicalReduction>3125</mechanicalReduction>
-	</actuator>
+    <type>transmission_interface/SimpleTransmission</type>
+    <joint name="joint5">
+      <hardwareInterface>hardware_interface/PositionJointInterface</hardwareInterface>
+    </joint>
+    <actuator name="motor5">
+      <mechanicalReduction>3125</mechanicalReduction>
+    </actuator>
   </transmission>
   <transmission name="tran6">
-	<type>transmission_interface/SimpleTransmission</type>
-	<joint name="joint6">
-	  <!--hardwareInterface>PositionJointInterface</hardwareInterface-->
-	  <!--hardwareInterface>VelocityJointInterface</hardwareInterface-->
-	  <hardwareInterface>EffortJointInterface</hardwareInterface>
-	</joint>
-	<actuator name="motor6">
-	  <!--hardwareInterface>PositionJointInterface</hardwareInterface-->
-	  <!--hardwareInterface>VelocityJointInterface</hardwareInterface-->
-	  <hardwareInterface>EffortJointInterface</hardwareInterface>
-	  <mechanicalReduction>3125</mechanicalReduction>
-	</actuator>
-  </transmission>
-  <!--this is silly, but need to include transmission spec in order to get ft_sensor link frame published-->
-  <transmission name="tran7">
-	<type>transmission_interface/SimpleTransmission</type>
-	<joint name="wrench_jnt">
-	  <!--hardwareInterface>PositionJointInterface</hardwareInterface-->
-	  <!--hardwareInterface>VelocityJointInterface</hardwareInterface-->
-	  <hardwareInterface>EffortJointInterface</hardwareInterface>
-	</joint>
-	<actuator name="motor7">
-	  <!--hardwareInterface>PositionJointInterface</hardwareInterface-->
-	  <!--hardwareInterface>VelocityJointInterface</hardwareInterface-->
-	  <hardwareInterface>EffortJointInterface</hardwareInterface>
-	  <mechanicalReduction>1</mechanicalReduction>
-	</actuator>
+    <type>transmission_interface/SimpleTransmission</type>
+    <joint name="joint6">
+      <hardwareInterface>hardware_interface/PositionJointInterface</hardwareInterface>
+    </joint>
+    <actuator name="motor6">
+      <mechanicalReduction>3125</mechanicalReduction>
+    </actuator>
+  </transmission>
+ <!--this is silly, but need to include transmission spec in order to get ft_sensor link frame published-->
+<transmission name="tran7">
+    <type>transmission_interface/SimpleTransmission</type>
+    <joint name="wrench_jnt">
+      <hardwareInterface>hardware_interface/PositionJointInterface</hardwareInterface>
+    </joint>
+    <actuator name="motor7">
+      <mechanicalReduction>1</mechanicalReduction>
+    </actuator>
   </transmission>
     <gazebo>
@@ -388,3 +348,14 @@
   </joint>
     <!-- Enable Joint Feedback -->
+    <gazebo reference="ft_sensor_jnt">
+        <provideFeedback>true</provideFeedback>
+    </gazebo>
+    <!-- The ft_sensor plugin -->
+    <gazebo>
+        <plugin name="ft_sensor" filename="libgazebo_ros_ft_sensor.so">
+            <updateRate>1000.0</updateRate>
+            <topicName>ft_sensor_topic</topicName>
+            <jointName>ft_sensor_jnt</jointName>
+        </plugin>
+    </gazebo>
 </robot>
